File: engineering/ELECTRONICS/M19O2_wiring/M19O2_wiring.sch (KiCad schematic (older format))
At the start: 30 parts, among them M1 ACDC_SMPS, M2 DCDC_Buck, M3 Arduino_Nano, M4 Relay_Board, M5 Compressor, M6 Fan, M7 Fan, M8 Fan, M9 Fan, P1 Wall_Plug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

Commit message: big push - added Hour Counter, and modified all renders and drawings
Parts:
- added H1: Hour_Counter, symbol M19O2_wiring:Hour_Counter
- M6: Field4 (none) -> COOLING FANS
- V4: value Contactor -> CONTACTOR; Field4 (none) -> [+]; Field5 (none) -> [-]; Field6 (none) -> 24 V DC
Connections:
- net GND: now also V4.1
- net at M1.+24V, M2.+24V, M4.COM1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: now also M4.COM4
- net at M5.L, S7.2: now also H1.L
- net at M5.N, S6.2: now also H1.N; no longer V4.2
- net at S2.2, S7.1: no longer M4.COM4
- net at M4.NO4: now also V4.2; no longer V4.1
- no-connect marks 24 -> 30
Other:
- note added: "Any Arduino Board\nor Compatible will\nwork here\n"
- note added: "Compressor\nContactor\nON / OFF"
- note added: "HOUR COUNTER\n(required to track\nmachine run time)"
- note added: "TEMP/HUMIDITY SENSOR - DHT22\nBUZZER\nPUSH BUTTON - COMPRESSOR\nLED RGB"
- note removed: "230V AC here !\nCan be avoided if you use\na 24V DC coil contactor"
- note removed: "Any Arduino Baord\nor Compatible will\nwork here\n"
- note removed: "Compressor\nON / OFF"
- note removed: "TEMP/HUMIDITY SENSOR\nBUZZER\nPUSH BUTTON\nLED RGB"

Commit message: some updates
Connections:
- net at F1.1, M1.L, S2.1: now also H1.L
- net at M1.N, S5.2, S6.1: now also H1.N
- net at M5.L, S7.2: now also H1.IN+; no longer H1.L
- net at M5.N, S6.2: now also H1.IN-; no longer H1.N
- no-connect marks 30 -> 28
Changed lines of the file:
@@
 	3200 1725 3200 2025
 Wire Wire Line
-	5450 3175 4175 3175
+	5450 3175 5200 3175
 Wire Wire Line
 	4175 3175 4175 1800
@@
 	4175 1800 4000 1800
 Wire Wire Line
-	5450 3475 3875 3475
+	5450 3475 5100 3475
 Wire Wire Line
 	3875 3475 3875 2100
@@
 NoConn ~ 4700 6925
 NoConn ~ 4800 6925
-NoConn ~ 4900 6925
-NoConn ~ 5000 6925
-Wire Wire Line
-	5200 6925 5200 6600
-Wire Wire Line
-	5200 6600 4175 6600
 Connection ~ 4175 6600
 Wire Wire Line
 	4175 6600 4175 6125
-Wire Wire Line
-	5100 6925 5100 6775
-Wire Wire Line
-	5100 6775 3875 6775
 Connection ~ 3875 6775
 Wire Wire Line
@@
 Text Notes 2925 7300 0    61   ~ 12
 HOUR COUNTER\n(required to track\nmachine run time)
+Wire Wire Line
+	4900 6925 4900 6775
+Wire Wire Line
+	4900 6775 3875 6775
+Wire Wire Line
+	5000 6925 5000 6600
+Wire Wire Line
+	5000 6600 4175 6600
+Wire Wire Line
+	5100 6925 5100 3475
+Connection ~ 5100 3475
+Wire Wire Line
+	5100 3475 3875 3475
+Wire Wire Line
+	5200 6925 5200 3175
+Connection ~ 5200 3175
+Wire Wire Line
+	5200 3175 4175 3175
 $EndSCHEMATC
