File: engineering/CAD/M19O2/M19O2_pneumatics_pictorial/M19O2_pneumatic_pictorial.sch (KiCad schematic (older format))
At the start: 0 parts

Commit message: documentation updates
Other:
- note removed: "Machined Aluminum or Brass\nOD to suit ID of pneumatic pipe\nOrifice bore dia = betn 1.0 to 1.2 mm\nLength, approx 10 mm or more\nAll edges deburred"
